File: Hardware/PCB_Satellogic/PCB_Satellogic.sch (KiCad schematic (older format))
At the start: 2 parts, among them U1 E22-900M30S_LoRa, U2 Node-MCU_ESP32_38PINES

Commit message: Introducción HW
Parts:
- added D?: 1N5819, Diode_THT:D_DO-41_SOD81_P10.16mm_Horizontal, symbol Diode:1N5819
Changed lines of the file:
@@
-EESchema Schematic File Version 4
-EELAYER 30 0
+EESchema Schematic File Version 5
+EELAYER 36 0
 EELAYER END
 $Descr A4 11693 8268
@@
 Comment3 ""
 Comment4 ""
+Comment5 ""
+Comment6 ""
+Comment7 ""
+Comment8 ""
+Comment9 ""
 $EndDescr
 $Comp
+L Diode:1N5819 D?
+U 1 1 00000000
+P 5800 3200
+F 0 "D?" H 5788 2950 50  0000 C CNN
+F 1 "1N5819" H 5788 3050 50  0000 C CNN
+F 2 "Diode_THT:D_DO-41_SOD81_P10.16mm_Horizontal" H 5800 3025 50  0001 C CNN
+F 3 "http://www.vishay.com/docs/88525/1n5817.pdf" H 5800 3200 50  0001 C CNN
+	1    5800 3200
+	-1   0    0    1
+$EndComp
+$Comp
 L Device:E22-900M30S_LoRa U1
