File: Hardware/PCB_Satellogic/PCB_Satellogic.kicad_pcb (KiCad board)
At the start: 2 copper layers, 92.7 x 78.7 mm, 2 parts, among them U1 E22-900M30S_LoRa, U2 Node-MCU_ESP32_38PINES

Commit message: Introducción HW
Parts:
- added D1: 1N5819, Diode_THT:D_DO-41_SOD81_P10.16mm_Horizontal, F.Cu at (121.9, 152.4)
- added U3: TP4065_Modulo_cargador_de_baterias, PCB_Satellogic:TP4056, F.Cu at (165.0, 147.4)
- moved U1 7.45 mm to (161.6, 117.0)
- moved U2 1.56 mm to (133.8, 121.7)
Connections:
- U1 pad 1: Net-(U1-Pad1) -> unconnected-(U1-Pad1)
- U1 pad 10: Net-(U1-Pad10) -> unconnected-(U1-Pad10)
- U1 pad 11: Net-(U1-Pad11) -> unconnected-(U1-Pad11)
- U1 pad 12: Net-(U1-Pad12) -> unconnected-(U1-Pad12)
- U1 pad 13: Net-(U1-Pad13) -> unconnected-(U1-Pad13)
- U1 pad 14: Net-(U1-Pad14) -> unconnected-(U1-Pad14)
- U1 pad 15: Net-(U1-Pad15) -> unconnected-(U1-Pad15)
- U1 pad 16: Net-(U1-Pad16) -> unconnected-(U1-Pad16)
- U1 pad 17: Net-(U1-Pad17) -> unconnected-(U1-Pad17)
- U1 pad 18: Net-(U1-Pad18) -> unconnected-(U1-Pad18)
- U1 pad 19: Net-(U1-Pad19) -> unconnected-(U1-Pad19)
- U1 pad 2: Net-(U1-Pad2) -> unconnected-(U1-Pad2)
- U1 pad 20: Net-(U1-Pad20) -> unconnected-(U1-Pad20)
- U1 pad 21: Net-(U1-Pad21) -> unconnected-(U1-Pad21)
- U1 pad 22: Net-(U1-Pad22) -> unconnected-(U1-Pad22)
- U1 pad 3: Net-(U1-Pad3) -> unconnected-(U1-Pad3)
- U1 pad 4: Net-(U1-Pad4) -> unconnected-(U1-Pad4)
- U1 pad 5: Net-(U1-Pad5) -> unconnected-(U1-Pad5)
- U1 pad 6: Net-(U1-Pad6) -> unconnected-(U1-Pad6)
- U1 pad 7: Net-(U1-Pad7) -> unconnected-(U1-Pad7)
- U1 pad 8: Net-(U1-Pad8) -> unconnected-(U1-Pad8)
- U1 pad 9: Net-(U1-Pad9) -> unconnected-(U1-Pad9)
- U2 pad 1: Net-(U2-Pad1) -> unconnected-(U2-Pad1)
- U2 pad 10: Net-(U2-Pad10) -> unconnected-(U2-Pad10)
- U2 pad 11: Net-(U2-Pad11) -> unconnected-(U2-Pad11)
- U2 pad 12: Net-(U2-Pad12) -> unconnected-(U2-Pad12)
- U2 pad 13: Net-(U2-Pad13) -> unconnected-(U2-Pad13)
- U2 pad 14: Net-(U2-Pad14) -> unconnected-(U2-Pad14)
- U2 pad 15: Net-(U2-Pad15) -> unconnected-(U2-Pad15)
- U2 pad 16: Net-(U2-Pad16) -> unconnected-(U2-Pad16)
- U2 pad 17: Net-(U2-Pad17) -> unconnected-(U2-Pad17)
- U2 pad 18: Net-(U2-Pad18) -> unconnected-(U2-Pad18)
- U2 pad 19: Net-(U2-Pad19) -> unconnected-(U2-Pad19)
- U2 pad 2: Net-(U2-Pad2) -> unconnected-(U2-Pad2)
- U2 pad 20: Net-(U2-Pad20) -> unconnected-(U2-Pad20)
- U2 pad 21: Net-(U2-Pad21) -> unconnected-(U2-Pad21)
- U2 pad 22: Net-(U2-Pad22) -> unconnected-(U2-Pad22)
- U2 pad 23: Net-(U2-Pad23) -> unconnected-(U2-Pad23)
- U2 pad 24: Net-(U2-Pad24) -> unconnected-(U2-Pad24)
- U2 pad 25: Net-(U2-Pad25) -> unconnected-(U2-Pad25)
- U2 pad 26: Net-(U2-Pad26) -> unconnected-(U2-Pad26)
- U2 pad 27: Net-(U2-Pad27) -> unconnected-(U2-Pad27)
- U2 pad 28: Net-(U2-Pad28) -> unconnected-(U2-Pad28)
- U2 pad 29: Net-(U2-Pad29) -> unconnected-(U2-Pad29)
- U2 pad 3: Net-(U2-Pad3) -> unconnected-(U2-Pad3)
- U2 pad 30: Net-(U2-Pad30) -> unconnected-(U2-Pad30)
- U2 pad 31: Net-(U2-Pad31) -> unconnected-(U2-Pad31)
- U2 pad 32: Net-(U2-Pad32) -> unconnected-(U2-Pad32)
- U2 pad 33: Net-(U2-Pad33) -> unconnected-(U2-Pad33)
- U2 pad 34: Net-(U2-Pad34) -> unconnected-(U2-Pad34)
- U2 pad 35: Net-(U2-Pad35) -> unconnected-(U2-Pad35)
- U2 pad 36: Net-(U2-Pad36) -> unconnected-(U2-Pad36)
- U2 pad 37: Net-(U2-Pad37) -> unconnected-(U2-Pad37)
- U2 pad 38: Net-(U2-Pad38) -> unconnected-(U2-Pad38)
- U2 pad 4: Net-(U2-Pad4) -> unconnected-(U2-Pad4)
- U2 pad 5: Net-(U2-Pad5) -> unconnected-(U2-Pad5)
- U2 pad 6: Net-(U2-Pad6) -> unconnected-(U2-Pad6)
- U2 pad 7: Net-(U2-Pad7) -> unconnected-(U2-Pad7)
- U2 pad 8: Net-(U2-Pad8) -> unconnected-(U2-Pad8)
- U2 pad 9: Net-(U2-Pad9) -> unconnected-(U2-Pad9)
Other:
- net class Default removed

Commit message: Introducción HW
Parts:
- moved U3 66.6 mm to (98.4, 146.1), turned to 90 degrees
- moved U1 15.2 mm to (170.2, 129.5)
- moved U2 12.9 mm to (133.4, 134.6)
- moved D1 8.03 mm to (114.3, 149.9), turned to 90 degrees
Other:
- board size 92.7 x 78.7 mm -> 105.1 x 62.6 mm

Commit message: Introducción HW
Parts:
- added 5V_out1: Conn_01x02, Connector_JST:JST_PH_B2B-PH-K_1x02_P2.00mm_Vertical, F.Cu at (106.7, 119.4)
- added BAT1: Conn_01x02, Connector_JST:JST_PH_B2B-PH-K_1x02_P2.00mm_Vertical, F.Cu at (94.5, 119.4)
- added U4: MT3608-Convertidor_Boost, PCB_Satellogic:MT3608-Convertidor_Boost, F.Cu at (86.4, 81.3)
- added UART2: Conn_01x02, Connector_JST:JST_PH_B2B-PH-K_1x02_P2.00mm_Vertical, F.Cu at (154.9, 120.7)
- U3: footprint PCB_Satellogic:TP4056 -> PCB_Satellogic:TP4056 - Módulo de carga de batería
- moved D1 43.3 mm to (111.8, 106.7), turned to 180 degrees
- moved U3 41.8 mm to (78.7, 109.2)
- moved U1 35.6 mm to (174.0, 94.1)
- moved U2 35.6 mm to (132.1, 99.1)
Connections:
- D1 pad 1: unconnected-(D1-K-Pad1) -> Net-(D1-K)
- D1 pad 2: unconnected-(D1-A-Pad2) -> /5V
- U1 pad 1: unconnected-(U1-GND-Pad1) -> /GND
- U1 pad 10: unconnected-(U1-Vcc-Pad10) -> /5V
- U1 pad 11: unconnected-(U1-GND-Pad11) -> /GND
- U1 pad 12: unconnected-(U1-GND-Pad12) -> /GND
- U1 pad 14: unconnected-(U1-BUSY-Pad14) -> /BUSY
- U1 pad 15: unconnected-(U1-NRST-Pad15) -> /RST_E22
- U1 pad 16: unconnected-(U1-MISO-Pad16) -> /MISO
- U1 pad 17: unconnected-(U1-MOSI-Pad17) -> /MOSI
- U1 pad 18: unconnected-(U1-SCK-Pad18) -> /SCK
- U1 pad 19: unconnected-(U1-NSS-Pad19) -> /NSS
- U1 pad 2: unconnected-(U1-GND-Pad2) -> /GND
- U1 pad 20: unconnected-(U1-GND-Pad20) -> /GND
- U1 pad 22: unconnected-(U1-GND-Pad22) -> /GND
- U1 pad 3: unconnected-(U1-GND-Pad3) -> /GND
- U1 pad 4: unconnected-(U1-GND-Pad4) -> /GND
- U1 pad 5: unconnected-(U1-GND-Pad5) -> /GND
- U1 pad 6: unconnected-(U1-RXEN-Pad6) -> /RXEN
- U1 pad 7: unconnected-(U1-TXEN-Pad7) -> /TXEN
- U1 pad 9: unconnected-(U1-Vcc-Pad9) -> /5V
- U2 pad 14: unconnected-(U2-GND-Pad14) -> /GND
- U2 pad 19: unconnected-(U2-Vin-Pad19) -> Net-(D1-K)
- U2 pad 27: unconnected-(U2-GPIO16-Pad27) -> /Rx2
- U2 pad 28: unconnected-(U2-GPIO17-Pad28) -> /Tx2
- U2 pad 29: unconnected-(U2-GPIO5-Pad29) -> /NSS
- U2 pad 30: unconnected-(U2-GPIO18-Pad30) -> /SCK
- U2 pad 31: unconnected-(U2-GPIO19-Pad31) -> /MISO
- U2 pad 33: unconnected-(U2-GPIO21-Pad33) -> /BUSY
- U2 pad 36: unconnected-(U2-GPIO22-Pad36) -> /RST_E22
- U2 pad 37: unconnected-(U2-GPIO23-Pad37) -> /MOSI
- U2 pad 38: unconnected-(U2-GND-Pad38) -> /GND
- U3 pad 3: unconnected-(U3-OUT--Pad3) -> Net-(U3-OUT-)
- U3 pad 4: unconnected-(U3-BAT--Pad4) -> /BAT-
- U3 pad 5: unconnected-(U3-BAT+-Pad5) -> /BAT+
- U3 pad 6: unconnected-(U3-OUT+-Pad6) -> Net-(U3-OUT+)
Routing:
- net /GND: track 0.00 -> 270.3 mm
- net /5V: track 0.00 -> 161.0 mm
- net /NSS: track 0.00 -> 93.9 mm
- net /SCK: track 0.00 -> 88.9 mm
- net /MISO: track 0.00 -> 81.3 mm
- net /MOSI: track 0.00 -> 80.6 mm
- net /RST_E22: track 0.00 -> 77.0 mm
- net /BUSY: track 0.00 -> 67.9 mm
- net /BAT+: track 0.00 -> 31.9 mm
- net /Rx2: track 0.00 -> 27.3 mm
- net /BAT-: track 0.00 -> 27.2 mm
- net /Tx2: track 0.00 -> 26.0 mm
- net Net-(U3-OUT-): track 0.00 -> 25.6 mm
- net Net-(D1-K): track 0.00 -> 20.4 mm
- net Net-(U3-OUT+): track 0.00 -> 13.3 mm
Other:
- board size 105.1 x 62.6 mm -> 128.3 x 53.3 mm
